File: P3_4x8x8_LED_Matrix_Clock/P3_4x8x8_LED_Matrix_Clock.kicad_sch (KiCad schematic)
At the start: 0 parts

Commit message: P3
Parts:
- added H1, H2, H3, H4: MountingHole, MountingHole:MountingHole_2.5mm, symbol Mechanical:MountingHole
- added J1: LED1_IN, Connector_PinHeader_2.54mm:PinHeader_1x05_P2.54mm_Vertical, symbol Connector:Conn_01x05_Pin
- added J2: Barrel_Jack, Connector_BarrelJack:BarrelJack_Horizontal, symbol Connector:Barrel_Jack
- added J3: LED1_OUT, Connector_PinSocket_2.54mm:PinSocket_1x05_P2.54mm_Vertical, symbol Connector:Conn_01x05_Pin
- added J4: LED2_IN, Connector_PinSocket_2.54mm:PinSocket_1x05_P2.54mm_Vertical, symbol Connector:Conn_01x05_Pin
- added J5: LED2_OUT, Connector_PinSocket_2.54mm:PinSocket_1x05_P2.54mm_Vertical, symbol Connector:Conn_01x05_Pin
- added J6: LED3_IN, Connector_PinSocket_2.54mm:PinSocket_1x05_P2.54mm_Vertical, symbol Connector:Conn_01x05_Pin
- added J7: LED3_OUT, Connector_PinSocket_2.54mm:PinSocket_1x05_P2.54mm_Vertical, symbol Connector:Conn_01x05_Pin
- added J8: LED4_IN, Connector_PinSocket_2.54mm:PinSocket_1x05_P2.54mm_Vertical, symbol Connector:Conn_01x05_Pin
- added J9: LED4_OUT, Connector_PinSocket_2.54mm:PinSocket_1x05_P2.54mm_Vertical, symbol Connector:Conn_01x05_Pin
- added R1, R2: 10K, Resistor_THT:R_Axial_DIN0204_L3.6mm_D1.6mm_P7.62mm_Horizontal, symbol Device:R
- added S1, S2: 1825967-1, Footprints_P3_Led_Matrix:SW_1825967-1, symbol Switch Tactile OFF (ON) SPST Round Button:1825967-1
- added S3: SS12D07VG4, Footprints_P3_Led_Matrix:SW_SS12D07VG4, symbol SS12D07VG4:SS12D07VG4
- added U1: ArduinoProMiniSimple, Footprints_P3_Led_Matrix:ArduinoProMiniCustom, symbol ArduinoProMiniSimple:ArduinoProMiniSimple
Connections:
- new net: J2.2, S3.3
- new net CLK0: J1.1 (Pin_1), U1.18 (13)
- new net CLK1: J3.1 (Pin_1)
- new net CLK2: J5.1 (Pin_1), J6.1 (Pin_1)
- new net CLK3: J7.1 (Pin_1), J8.1 (Pin_1)
- new net CS0: J1.2 (Pin_2), U1.15 (10)
- new net CS1: J3.2 (Pin_2), J4.2 (Pin_2)
- new net CS2: J5.2 (Pin_2), J6.2 (Pin_2)
- new net CS3: J7.2 (Pin_2), J8.2 (Pin_2)
- new net DIN0: J1.3 (Pin_3), U1.16 (11)
- new net DIN1: J3.3 (Pin_3), J4.3 (Pin_3)
- new net DIN2: J5.3 (Pin_3), J6.3 (Pin_3)
- new net DIN3: J7.3 (Pin_3), J8.3 (Pin_3)
- new net GND: J1.4 (Pin_4), J3.4 (Pin_4), J4.4 (Pin_4), J5.4 (Pin_4), J6.4 (Pin_4), J7.4 (Pin_4), J8.4 (Pin_4), R1.2, R2.2, S3.2, U1.12 (GND), U1.25 (GND), U1.27 (GND), U1.28 (GND), U1.3 (GND)
- new net MODE_SELECT: R2.1, S2.1, S2.2, U1.6 (4)
- new net TIMER_RESET: R1.1, S1.1, S1.2, U1.7 (5)
- new net VCC: J1.5 (Pin_5), J2.1, J3.5 (Pin_5), J4.5 (Pin_5), J5.5 (Pin_5), J6.5 (Pin_5), J7.5 (Pin_5), J8.5 (Pin_5), S1.3, S1.4, S2.3, S2.4, U1.29 (VCC)
- no-connect marks 0 -> 32
